Commit message: fixed robot not move issue

File: urdf/drive_bot.xacro (robot description, xacro)
@@ -31,6 +31,18 @@
       </geometry>
     </visual>
+    <collision name='back_caster_collision'>
+      <origin xyz="-0.25 0 -0.05" rpy=" 0 0 0"/>
+      <geometry>
+        <sphere radius="0.0499"/>
+      </geometry>
+    </collision>
+    <visual name='back_caster_visual'>
+      <origin xyz="-0.25 0 -0.05" rpy=" 0 0 0"/>
+      <geometry>
+        <sphere radius="0.05"/>
+      </geometry>
+    </visual>
     <collision name='front_caster_collision'>
-      <origin xyz="0.2 0 -0.05" rpy=" 0 0 0"/>
+      <origin xyz="0.25 0 -0.05" rpy=" 0 0 0"/>
       <geometry>
         <sphere radius="0.0499"/>
@@ -38,5 +50,5 @@
     </collision>
     <visual name='front_caster_visual'>
-      <origin xyz="0.2 0 -0.05" rpy=" 0 0 0"/>
+      <origin xyz="0.25 0 -0.05" rpy=" 0 0 0"/>
       <geometry>
         <sphere radius="0.05"/>
@@ -125,5 +137,5 @@
     <dynamics damping="1.0" friction="1.0"/>
   </joint>
-  <link name='left_wheel'>
+  <link name='rear_left_wheel'>
     <inertial>
       <mass value="2.0"/>
@@ -135,18 +147,18 @@
       />
     </inertial>
-    <collision name='left_wheel_collision'>
-      <origin xyz="0 0 0" rpy="0 1.5707 1.5707"/>
-      <geometry>
-        <cylinder radius="0.2" length="0.05"/>
-      </geometry>
-    </collision>
-    <visual name='left_wheel_visual'>
-      <origin xyz="0 0 0" rpy="0 1.5707 1.5707"/>
-      <geometry>
-        <cylinder radius="0.2" length="0.05"/>
-      </geometry>
-    </visual>
-  </link>
-  <link name='right_wheel'>
+    <collision name='rear_left_wheel_collision'>
+      <origin xyz="0 0 0" rpy="0 1.5707 1.5707"/>
+      <geometry>
+        <cylinder radius="0.15" length="0.1"/>
+      </geometry>
+    </collision>
+    <visual name='rear_left_wheel_visual'>
+      <origin xyz="0 0 0" rpy="0 1.5707 1.5707"/>
+      <geometry>
+        <cylinder radius="0.15" length="0.1"/>
+      </geometry>
+    </visual>
+  </link>
+  <link name='rear_right_wheel'>
     <inertial>
       <mass value="2.0"/>
@@ -158,14 +170,14 @@
       />
     </inertial>
-    <collision name='right_wheel_collision'>
-      <origin xyz="0 0 0" rpy="0 1.5707 1.5707"/>
-      <geometry>
-        <cylinder radius="0.2" length="0.05"/>
-      </geometry>
-    </collision>
-    <visual name='right_wheel_visual'>
+    <collision name='rear_right_wheel_collision'>
+      <origin xyz="0 0 0" rpy="0 1.5707 1.5707"/>
+      <geometry>
+        <cylinder radius="0.15" length="0.1"/>
+      </geometry>
+    </collision>
+    <visual name='rear_right_wheel_visual'>
       <origin xyz="0 0 0" rpy=" 0 1.5707 1.5707"/>
       <geometry>
-        <cylinder radius="0.2" length="0.05"/>
+        <cylinder radius="0.15" length="0.1"/>
       </geometry>
     </visual>
@@ -220,7 +232,7 @@
     </visual>
   </link>
-  <joint type="continuous" name="left_wheel_hinge">
-    <origin xyz="-0.15 0.2 0.1" rpy="0 0 0"/>
-    <child link="left_wheel"/>
+  <joint type="continuous" name="rear_left_wheel_hinge">
+    <origin xyz="0 0.25 0.05" rpy="0 0 0"/>
+    <child link="rear_left_wheel"/>
     <parent link="chassis"/>
     <axis xyz="0 1 0" rpy="0 0 0"/>
@@ -228,7 +240,7 @@
     <dynamics damping="1.0" friction="1.0"/>
   </joint>
-  <joint type="continuous" name="right_wheel_hinge">
-    <origin xyz="-0.15 -0.2 0.1" rpy="0 0 0"/>
-    <child link="right_wheel"/>
+  <joint type="continuous" name="rear_right_wheel_hinge">
+    <origin xyz="0 -0.25 0.05" rpy="0 0 0"/>
+    <child link="rear_right_wheel"/>
     <parent link="chassis"/>
     <axis xyz="0 1 0" rpy="0 0 0"/>

Commit message: Update drive_bot URDF
Corrected the path of the lidar model

File: urdf/drive_bot.xacro (robot description, xacro)
@@ -228,5 +228,5 @@
       <origin xyz="0 0 0" rpy=" 0 0 0"/>
       <geometry>
-        <mesh filename = "package://my_robot/meshes/hokuyo.dae"/>
+        <mesh filename = "package://drive_bot/meshes/hokuyo.dae"/>
       </geometry>
     </visual>

Commit message: finish project

File: urdf/drive_bot.xacro (robot description, xacro)
@@ -183,5 +183,5 @@
     </visual>
   </link>
-  <link name='camera'>
+  <link name='camera_link'>
     <inertial>
       <mass value="2"/>
@@ -193,5 +193,5 @@
       />
     </inertial>
-    <collision name='camera_collision'>
+    <collision name='camera_link_collision'>
       <origin xyz="0 0 0" rpy="0 0 0"/>
       <geometry>
@@ -199,5 +199,5 @@
       </geometry>
     </collision>
-    <visual name='camera_visual'>
+    <visual name='camera_link_visual'>
       <origin xyz="0 0 0" rpy=" 0 0 0"/>
       <geometry>
@@ -205,4 +205,11 @@
       </geometry>
     </visual>
+  </link>
+  <joint name="camera_optical_joint" type="fixed">
+    <origin xyz="0 0 0" rpy="-1.5707 0 -1.5707"/>
+    <parent link="camera_link"/>
+    <child link="camera_link_optical"/>
+  </joint>
+  <link name="camera_link_optical">
   </link>
   <gazebo reference="camera">
@@ -250,5 +257,5 @@
   <joint type="fixed" name="camera_joint">
     <origin xyz="0.275 0 0.04" rpy="0 0 0"/>
-    <child link="camera"/>
+    <child link="camera_link"/>
     <parent link="chassis"/>
     <axis xyz="0 1 0" rpy="0 0 0"/>
